File: KiCad/Projet/Projet.kicad_pcb (KiCad board)
At the start: 2 copper layers, 68.6 x 53.3 mm, 8 parts, among them P1 Power, P2 Analog, P3 Digital, P4 Digital, P5 CONN_01X01, P6 CONN_01X01, P7 CONN_01X01, P8 CONN_01X01

Commit message: Modification sch + Placements pcb
Parts:
- added ?: , , F.Cu at (144.0, 107.3)
- added C1: CP_Radial_Tantal_D5.5mm_P5.00mm, Capacitor_THT:CP_Radial_Tantal_D5.5mm_P5.00mm, F.Cu at (147.8, 113.7)
- added C2: CP_Radial_Tantal_D5.5mm_P5.00mm, Capacitor_THT:CP_Radial_Tantal_D5.5mm_P5.00mm, F.Cu at (163.1, 97.2)
- added C3: CP_Radial_Tantal_D5.5mm_P5.00mm, Capacitor_THT:CP_Radial_Tantal_D5.5mm_P5.00mm, F.Cu at (163.1, 106.0)
- added C4: CP_Radial_Tantal_D5.5mm_P5.00mm, Capacitor_THT:CP_Radial_Tantal_D5.5mm_P5.00mm, F.Cu at (163.1, 114.9)
- added R1: R_Axial_DIN0207_L6.3mm_D2.5mm_P10.16mm_Horizontal, Resistor_THT:R_Axial_DIN0207_L6.3mm_D2.5mm_P10.16mm_Horizontal, F.Cu at (128.8, 98.4)
- added R2: R_Axial_DIN0207_L6.3mm_D2.5mm_P10.16mm_Horizontal, Resistor_THT:R_Axial_DIN0207_L6.3mm_D2.5mm_P10.16mm_Horizontal, F.Cu at (128.8, 104.8)
- added R3: R_Axial_DIN0207_L6.3mm_D2.5mm_P10.16mm_Horizontal, Resistor_THT:R_Axial_DIN0207_L6.3mm_D2.5mm_P10.16mm_Horizontal, F.Cu at (128.8, 111.1)
- added R4: R_Axial_DIN0207_L6.3mm_D2.5mm_P10.16mm_Horizontal, Resistor_THT:R_Axial_DIN0207_L6.3mm_D2.5mm_P10.16mm_Horizontal, F.Cu at (128.8, 117.5)
- added R5: R_Axial_DIN0207_L6.3mm_D2.5mm_P10.16mm_Horizontal, Resistor_THT:R_Axial_DIN0207_L6.3mm_D2.5mm_P10.16mm_Horizontal, F.Cu at (145.3, 98.4)
- added R6: R_Axial_DIN0207_L6.3mm_D2.5mm_P10.16mm_Horizontal, Resistor_THT:R_Axial_DIN0207_L6.3mm_D2.5mm_P10.16mm_Horizontal, F.Cu at (145.3, 104.8)
- added S1: TO-5-10_Window, Empreinte_Capteur_Gaz:Empreinte_Capteur_Gaz, F.Cu at (133.9, 85.7)
- added U1: RN2483_breakout, Empreinte_RN2483:RN2483_breakout, F.Cu at (116.1, 111.1)
- added U2: DIP-8_W7.62mm_LongPads, Empreinte_LTC1050:Package_DIP-8_W7.62mm_LongPads, F.Cu at (152.9, 81.9)
