File: KiCad/Projet/Projet.kicad_pcb (KiCad board)
At the start: 2 copper layers, 68.6 x 53.3 mm, 22 parts, among them P1 Power, P2 Analog, P3 Digital, P4 Digital, P5 CONN_01X01, P6 CONN_01X01, P7 CONN_01X01, P8 CONN_01X01, U1 RN2483_breakout, U2 DIP-8_W7.62mm_LongPads

Commit message: V1 PCB + readme
Parts:
- moved R4 33.2 mm to (161.8, 113.7)
- moved R3 19.2 mm to (147.8, 113.7)
- moved R5 14.0 mm to (131.3, 98.4)
- moved C2 13.3 mm to (166.9, 84.5)
- moved C3 13.3 mm to (166.9, 93.3)
- moved R1 12.8 mm to (130.0, 111.1)
- moved R2 12.8 mm to (130.0, 117.5)
- moved C4 10.2 mm to (161.8, 104.8)
- moved R6 10.2 mm to (135.1, 104.8)
- moved C1 9.67 mm to (151.6, 104.8)
- moved S1 4.02 mm to (137.7, 84.5), turned to 270 degrees
- moved U2 2.54 mm to (152.9, 84.5)
Connections:
- C1 pad 2: (no net) -> GND
- C2 pad 2: (no net) -> GND
- C3 pad 1: (no net) -> +5V
- C3 pad 2: (no net) -> GND
- R1 pad 2: (no net) -> GND
- R2 pad 2: (no net) -> GND
- R6 pad 1: (no net) -> +5V
- S1 pad 10: (no net) -> GND
- S1 pad 2: (no net) -> +5V
- S1 pad 3: (no net) -> +5V
- S1 pad 5: (no net) -> GND
- S1 pad 6: (no net) -> GND
- S1 pad 8: (no net) -> GND
- U1 pad 8: (no net) -> GND
- U2 pad 7: (no net) -> +5V
Routing:
- net (no net): track 0.00 -> 480.1 mm
- net +3V3: track 0.00 -> 49.0 mm
- net +5V: track 0.00 -> 8.98 mm
- net /7: track 0.00 -> 1.27 mm
- net /A1: track 0.00 -> 0.89 mm
- added copper zone on F.Cu, net +5V
- added copper zone on B.Cu, net GND
Other:
- board text added: "Opétatereurs: Baptiste Mennesson Brice Moutanin"
